File: FrontDoorController.sch (EAGLE design)
At the start: 11 parts

Commit message: Door_Control_PCB: Add SW3 and SW4 from Lockitron
The Lockitron has 4 limit switches instead of 2 like I originally
thought.  They also need a common place to wire their NC connections to
and with this many switches it seemed best to give them their own header
row, causing some other components to have to move and some other pins
to need moving as well.  Things all seem to flow well now and there
should be plenty of power to all of the components.
Parts:
- removed R1: 1K, SparkFun-Resistors:RESISTOR0603
- added JP2: (no value), SparkFun-Connectors:M04LOCK
Connections:
- removed net A0: PHOTONG$1.A0, U$3.A0
- removed net A1: PHOTONG$1.A1, U$3.A1
- removed net VM: C1.+, C2.1, D1.A, JP1.6, U$2.VM1, U$2.VM2, U$2.VM3
- new net SW3: JP2.1, PHOTONG$1.A0, U$3.A0
- new net SW4: JP2.2, PHOTONG$1.A1, U$3.A1
- new net VBAK: PHOTONG$1.VBAT, U$3.VBAT
- net DOORSW: no longer R1.2
- net GND: now also JP1.8, JP1.9; no longer R1.1
- net SW1: now also JP2.3; no longer JP1.8
- net SW2: now also JP2.4; no longer JP1.9
- net VBAT: now also C1.+, C2.1, D1.A, JP1.6, U$2.VM1, U$2.VM2, U$2.VM3; no longer PHOTONG$1.VBAT, U$3.VBAT
Other:
- note added: "Other Limit switches from Lockitron"
- note added: "VBAT from AA Batts"
- note removed: "3V3 -> Reed SW -> DOORSW -> Photon Pin"
- note removed: "VM from AA Batts"
- note removed: "|-> 1K Ohm -> GND"
Changed lines of the file:
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@@
 <part name="D1" library="SparkFun-DiscreteSemi" deviceset="DIODE" device="PTH"/>
 <part name="U$3" library="Mikes-Stuff" deviceset="PHOTON" device="_WITH_HEADERS"/>
-<part name="R1" library="SparkFun-Resistors" deviceset="RESISTOR" device="0603" value="1K"/>
 <part name="U$1" library="Mikes-Stuff" deviceset="SPARK_LOGO" device="LARGE"/>
+<part name="JP2" library="SparkFun-Connectors" deviceset="M04" device="LOCK"/>
 </parts>
 <sheets>
 <sheet>
 <plain>
-<text x="139.7" y="158.75" size="1.778" layer="91">VM from AA Batts</text>
+<text x="139.7" y="158.75" size="1.778" layer="91">VBAT from AA Batts</text>
 <text x="123.825" y="102.235" size="1.778" layer="91">0.6V drop, makes ~6V closer to ~5V</text>
 <text x="6.35" y="47.625" size="1.778" layer="91">This is an overlay for the Photon through-hole pins for prototyping purposes</text>
 <text x="143.51" y="162.56" size="1.778" layer="91">Limit switches
 from Lockitron</text>
-<text x="93.98" y="137.16" size="1.778" layer="91">3V3 -&gt; Reed SW -&gt; DOORSW -&gt; Photon Pin</text>
-<text x="114.3" y="134.62" size="1.778" layer="91">|-&gt; 1K Ohm -&gt; GND</text>
+<text x="138.43" y="127" size="1.778" layer="91">Other Limit switches
+from Lockitron</text>
 </plain>
 <instances>
@@
 </instance>
 <instance part="U$3" gate="G$1" x="30.48" y="81.153"/>
-<instance part="R1" gate="G$1" x="119.38" y="127"/>
 <instance part="U$1" gate="G$1" x="15.24" y="38.1"/>
+<instance part="JP2" gate="G$1" x="166.37" y="127"/>
 </instances>
 <busses>
@@
 </segment>
 <segment>
-<pinref part="R1" gate="G$1" pin="1"/>
-<wire x1="114.3" y1="127" x2="109.728" y2="127" width="0.1524" layer="91"/>
-<label x="110.236" y="127" size="1.778" layer="95"/>
-</segment>
-<segment>
 <pinref part="JP1" gate="G$1" pin="5"/>
 <wire x1="170.815" y1="154.94" x2="174.8536" y2="154.94" width="0.1524" layer="91"/>
 <label x="170.815" y="154.94" size="1.778" layer="95"/>
 </segment>
+<segment>
+<pinref part="JP1" gate="G$1" pin="9"/>
+<wire x1="170.815" y1="165.1" x2="174.625" y2="165.1" width="0.1524" layer="91"/>
+<label x="170.815" y="165.1" size="1.778" layer="95"/>
+</segment>
+<segment>
+<pinref part="JP1" gate="G$1" pin="8"/>
+<wire x1="170.815" y1="162.56" x2="174.5742" y2="162.56" width="0.1524" layer="91"/>
+<label x="170.8404" y="162.56" size="1.778" layer="95"/>
+</segment>
 </net>
 <net name="TX" class="0">
@@
 <wire x1="12.7" y1="63.373" x2="7.62" y2="63.373" width="0.1524" layer="91"/>
 <label x="7.62" y="63.373" size="1.778" layer="95"/>
-</segment>
-</net>
-<net name="A1" class="0">
-<segment>
-<pinref part="PHOTON" gate="G$1" pin="A1"/>
-<wire x1="12.7" y1="126.238" x2="7.62" y2="126.238" width="0.1524" layer="91"/>
-<label x="7.62" y="126.238" size="1.778" layer="95"/>
-</segment>
-<segment>
-<pinref part="U$3" gate="G$1" pin="A1"/>
-<wire x1="12.7" y1="58.293" x2="7.62" y2="58.293" width="0.1524" layer="91"/>
-<label x="7.62" y="58.293" size="1.778" layer="95"/>
-</segment>
-</net>
-<net name="A0" class="0">
-<segment>
-<pinref part="PHOTON" gate="G$1" pin="A0"/>
-<wire x1="12.7" y1="121.158" x2="7.62" y2="121.158" width="0.1524" layer="91"/>
-<label x="7.62" y="121.158" size="1.778" layer="95"/>
-</segment>
-<segment>
-<pinref part="U$3" gate="G$1" pin="A0"/>
-<wire x1="12.7" y1="53.213" x2="7.62" y2="53.213" width="0.1524" layer="91"/>
-<label x="7.62" y="53.213" size="1.778" layer="95"/>
 </segment>
 </net>
@@
 </segment>
 </net>
-<net name="VM" class="0">
+<net name="VBAT" class="0">
 <segment>
 <pinref part="U$2" gate="G$1" pin="VM1"/>
@@
 </segment>
 </net>
-<net name="VBAT" class="0">
+<net name="VBAK" class="0">
 <segment>
 <pinref part="PHOTON" gate="G$1" pin="VBAT"/>
@@
 <net name="SW1" class="0">
 <segment>
-<pinref part="JP1" gate="G$1" pin="8"/>
-<wire x1="170.815" y1="162.56" x2="174.625" y2="162.56" width="0.1524" layer="91"/>
-<label x="170.815" y="162.56" size="1.778" layer="95"/>
-</segment>
-<segment>
 <pinref part="PHOTON" gate="G$1" pin="D0"/>
 <wire x1="48.26" y1="121.158" x2="53.34" y2="121.158" width="0.1524" layer="91"/>
@@
 <label x="48.26" y="53.213" size="1.778" layer="95"/>
 </segment>
+<segment>
+<pinref part="JP2" gate="G$1" pin="3"/>
+<wire x1="171.45" y1="129.54" x2="175.26" y2="129.54" width="0.1524" layer="91"/>
+<label x="171.45" y="129.54" size="1.778" layer="95"/>
+</segment>
 </net>
 <net name="SW2" class="0">
-<segment>
-<pinref part="JP1" gate="G$1" pin="9"/>
-<wire x1="170.815" y1="165.1" x2="174.625" y2="165.1" width="0.1524" layer="91"/>
-<label x="170.815" y="165.1" size="1.778" layer="95"/>
-</segment>
 <segment>
 <pinref part="PHOTON" gate="G$1" pin="D1"/>
@@
 <label x="48.26" y="58.293" size="1.778" layer="95"/>
 </segment>
+<segment>
+<pinref part="JP2" gate="G$1" pin="4"/>
+<wire x1="171.45" y1="132.08" x2="175.26" y2="132.08" width="0.1524" layer="91"/>
+<label x="171.45" y="132.08" size="1.778" layer="95"/>
+</segment>
 </net>
 <net name="DOORSW" class="0">
@@
 <label x="48.26" y="63.373" size="1.778" layer="95"/>
 </segment>
-<segment>
-<pinref part="R1" gate="G$1" pin="2"/>
-<wire x1="124.46" y1="127" x2="128.778" y2="127" width="0.1524" layer="91"/>
-<label x="124.714" y="127" size="1.778" layer="95"/>
-</segment>
-</net>
+</net>
+<net name="SW4" class="0">
+<segment>
+<pinref part="JP2" gate="G$1" pin="2"/>
+<wire x1="171.45" y1="127" x2="175.26" y2="127" width="0.1524" layer="91"/>
+<label x="171.45" y="127" size="1.778" layer="95"/>
+</segment>
+<segment>
+<pinref part="PHOTON" gate="G$1" pin="A1"/>
+<wire x1="12.7" y1="126.238" x2="7.62" y2="126.238" width="0.1524" layer="91"/>
+<label x="7.62" y="126.238" size="1.778" layer="95"/>
+</segment>
+<segment>
+<pinref part="U$3" gate="G$1" pin="A1"/>
+<wire x1="12.7" y1="58.293" x2="7.62" y2="58.293" width="0.1524" layer="91"/>
+<label x="7.62" y="58.293" size="1.778" layer="95"/>
+</segment>
+</net>
+<net name="SW3" class="0">
+<segment>
+<pinref part="JP2" gate="G$1" pin="1"/>
+<wire x1="171.45" y1="124.46" x2="175.26" y2="124.46" width="0.1524" layer="91"/>
+<label x="171.45" y="124.46" size="1.778" layer="95"/>
+</segment>
+<segment>
+<pinref part="PHOTON" gate="G$1" pin="A0"/>
+<wire x1="12.7" y1="121.158" x2="7.62" y2="121.158" width="0.1524" layer="91"/>
+<label x="7.62" y="121.158" size="1.778" layer="95"/>
+</segment>
+<segment>
+<pinref part="U$3" gate="G$1" pin="A0"/>
+<wire x1="12.7" y1="53.213" x2="7.62" y2="53.213" width="0.1524" layer="91"/>
+<label x="7.62" y="53.213" size="1.778" layer="95"/>
+</segment>
+</net>
